Commit message: update

File: FR5_V6/urdf/FR5_V6.urdf (robot description, URDF)
Before this commit: robot FR5_V6, 7 links, 6 joints
Joints:
- removed joint Joint1
- removed joint Joint2
- removed joint Joint3
- removed joint Joint4
- removed joint Joint5
- removed joint Joint6
- added joint elbow_joint: type revolute, parent FR5_link2, child FR5_link3, origin xyz=-0.425 0 0 rpy=0 0 0, axis 0 0 1, limit lower=-3.1415 upper=3.1415 effort=0 velocity=3.14
- added joint shoulder_lift_joint: type revolute, parent FR5_link1, child FR5_link2, origin xyz=0 0 0 rpy=1.5708 0 0, axis 0 0 1, limit lower=-4.712 upper=1.57 effort=0 velocity=2.1
- added joint shoulder_pan_joint: type revolute, parent FR5_base_link, child FR5_link1, origin xyz=0 0 0.152 rpy=0 0 0, axis 0 0 1, limit lower=-3.1415 upper=3.1415 effort=0 velocity=2.1
- added joint wrist_1_joint: type revolute, parent FR5_link3, child FR5_link4, origin xyz=-0.395 0 0.102 rpy=0 0 0, axis 0 0 1, limit lower=-4.712 upper=1.57 effort=0 velocity=2.1
- added joint wrist_2_joint: type revolute, parent FR5_link4, child FR5_link5, origin xyz=0 -0.102 0 rpy=1.5708 0 0, axis 0 0 1, limit lower=-3.1415 upper=3.1415 effort=0 velocity=2.1
- added joint wrist_3_joint: type revolute, parent FR5_link5, child FR5_link6, origin xyz=0 0.1 0 rpy=-1.5708 0 0, axis 0 0 1, limit lower=-3.1415 upper=3.1415 effort=0 velocity=2.1

File: FR5_V6/urdf/FR5_V6_RTQ85.urdf (robot description, URDF)
Before this commit: robot FR5_V6, 19 links, 18 joints
Links:
- removed link robotiq_85_base_link
- removed link robotiq_85_left_finger_link
- removed link robotiq_85_left_finger_tip_link
- removed link robotiq_85_left_inner_knuckle_link
- removed link robotiq_85_left_knuckle_link
- removed link robotiq_85_right_finger_link
- removed link robotiq_85_right_finger_tip_link
- removed link robotiq_85_right_inner_knuckle_link
- removed link robotiq_85_right_knuckle_link
- added link left_inner_finger, mass 0.019555; collision mesh filename=package://FR5_V6/meshes/rtq85/collision/robotiq_85_finger_t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; visual mesh filename=package://FR5_V6/meshes/rtq85/visual/robotiq_85_finger_tip_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
- added link left_inner_knuckle, mass 0.029951; collision mesh filename=package://FR5_V6/meshes/rtq85/collision/robotiq_85_inner_kn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; visual mesh filename=package://FR5_V6/meshes/rtq85/visual/robotiq_85_inner_knuck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
- added link left_outer_finger, mass 0.027309; collision mesh filename=package://FR5_V6/meshes/rtq85/collision/robotiq_85_finger_l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; visual mesh filename=package://FR5_V6/meshes/rtq85/visual/robotiq_85_finger_link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
- added link left_outer_knuckle, mass 0.018491; collision mesh filename=package://FR5_V6/meshes/rtq85/collision/robotiq_85_outer_kn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; visual mesh filename=package://FR5_V6/meshes/rtq85/visual/robotiq_85_outer_knuck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
- added link right_inner_finger, mass 0.019555; collision mesh filename=package://FR5_V6/meshes/rtq85/collision/robotiq_85_finger_t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; visual mesh filename=package://FR5_V6/meshes/rtq85/visual/robotiq_85_finger_tip_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
- added link right_inner_knuckle, mass 0.029951; collision mesh filename=package://FR5_V6/meshes/rtq85/collision/robotiq_85_inner_kn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; visual mesh filename=package://FR5_V6/meshes/rtq85/visual/robotiq_85_inner_knuck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
- added link right_outer_finger, mass 0.027309; collision mesh filename=package://FR5_V6/meshes/rtq85/collision/robotiq_85_finger_l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; visual mesh filename=package://FR5_V6/meshes/rtq85/visual/robotiq_85_finger_link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
- added link right_outer_knuckle, mass 0.018491; collision mesh filename=package://FR5_V6/meshes/rtq85/collision/robotiq_85_outer_kn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; visual mesh filename=package://FR5_V6/meshes/rtq85/visual/robotiq_85_outer_knuck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
- added link robotiq_base_link, mass 0.636951; collision mesh filename=package://FR5_V6/meshes/rtq85/collision/robotiq_85_base_lin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; visual mesh filename=package://FR5_V6/meshes/rtq85/visual/robotiq_85_base_link.d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
Joints:
- removed joint robotiq_85_left_finger_joint
- removed joint robotiq_85_left_finger_tip_joint
- removed joint robotiq_85_left_inner_knuckle_joint
- removed joint robotiq_85_left_knuckle_joint
- removed joint robotiq_85_right_finger_joint
- removed joint robotiq_85_right_finger_tip_joint
- removed joint robotiq_85_right_inner_knuckle_joint
- removed joint robotiq_85_right_knuckle_joint
- added joint finger_joint: type revolute, parent robotiq_base_link, child left_outer_knuckle, origin xyz=0.05490451627 0.03060114443 0.0 rpy=3.141592653589793 0.0 0.0, axis 0 0 1, limit lower=0.0 upper=0.804 effort=1000 velocity=2.0
- added joint left_inner_finger_joint: type revolute, parent left_inner_knuckle, child left_inner_finger, origin xyz=0.04303959807 -0.03759940821 0.0 rpy=0.0 0.0 0.0, axis 0 0 1, limit lower=-3.14 upper=3.14 effort=0.1 velocity=100.0, mimic joint=finger_joint multiplier=-1 offset=0
- added joint left_inner_knuckle_joint: type revolute, parent robotiq_base_link, child left_inner_knuckle, origin xyz=0.06142 0.0127 0 rpy=3.141592653589793 0.0 0.0, axis 0 0 1, limit lower=-3.14 upper=3.14 effort=0.1 velocity=100.0, mimic joint=finger_joint multiplier=1 offset=0
- added joint left_outer_finger_joint: type fixed, parent left_outer_knuckle, child left_outer_finger, origin xyz=-0.00408552455 -0.03148604435 0.0 rpy=0 0 0
- added joint right_inner_finger_joint: type revolute, parent right_inner_knuckle, child right_inner_finger, origin xyz=0.04303959807 -0.03759940821  0.0 rpy=0.0 0.0 0.0, axis 0 0 1, limit lower=-3.14 upper=3.14 effort=0.1 velocity=100.0, mimic joint=finger_joint multiplier=-1 offset=0
- added joint right_inner_knuckle_joint: type revolute, parent robotiq_base_link, child right_inner_knuckle, origin xyz=0.06142 -0.0127 0 rpy=0 0 0, axis 0 0 1, limit lower=-3.14 upper=3.14 effort=0.1 velocity=100.0, mimic joint=finger_joint multiplier=1 offset=0
- added joint right_outer_finger_joint: type fixed, parent right_outer_knuckle, child right_outer_finger, origin xyz=-0.00408552455 -0.03148604435 0.0 rpy=0 0 0
- added joint right_outer_knuckle_joint: type revolute, parent robotiq_base_link, child right_outer_knuckle, origin xyz=0.05490451627 -0.03060114443 0.0 rpy=0.0 0.0 0.0, axis 0 0 1, limit lower=-3.14 upper=3.14 effort=1000 velocity=100.0, mimic joint=finger_joint multiplier=1 offset=0
- joint robotiq_85_base_joint: child robotiq_85_base_link -> robotiq_base_link

File: FR5_V6/urdf/FR5_V6_WSG50.urdf (robot description, URDF)
Before this commit: robot FR5_V6_WSG50, 11 links, 10 joints
Links:
- link FR5_base_link: geometry collision mesh filename=/home/yan/Documents/isaacsim_usd/FR5_V6/meshes/fr5_wsg50/FR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 scale=1. 1. 1.; visual mesh filename=/home/yan/Documents/isaacsim_usd/FR5_V6/meshes/fr5_wsg50/FR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 scale=1. 1. 1.
- link FR5_link1: geometry collision mesh filename=/home/yan/Documents/isaacsim_usd/FR5_V6/meshes/fr5_wsg50/FR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 scale=1. 1. 1.; visual mesh filename=/home/yan/Documents/isaacsim_usd/FR5_V6/meshes/fr5_wsg50/FR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 scale=1. 1. 1.
- link FR5_link2: geometry collision mesh filename=/home/yan/Documents/isaacsim_usd/FR5_V6/meshes/fr5_wsg50/FR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 scale=1. 1. 1.; visual mesh filename=/home/yan/Documents/isaacsim_usd/FR5_V6/meshes/fr5_wsg50/FR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 scale=1. 1. 1.
- link FR5_link3: geometry collision mesh filename=/home/yan/Documents/isaacsim_usd/FR5_V6/meshes/fr5_wsg50/FR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 scale=1. 1. 1.; visual mesh filename=/home/yan/Documents/isaacsim_usd/FR5_V6/meshes/fr5_wsg50/FR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 scale=1. 1. 1.
- link FR5_link4: geometry collision mesh filename=/home/yan/Documents/isaacsim_usd/FR5_V6/meshes/fr5_wsg50/FR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 scale=1. 1. 1.; visual mesh filename=/home/yan/Documents/isaacsim_usd/FR5_V6/meshes/fr5_wsg50/FR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 scale=1. 1. 1.
- link FR5_link5: geometry collision mesh filename=/home/yan/Documents/isaacsim_usd/FR5_V6/meshes/fr5_wsg50/FR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 scale=1. 1. 1.; visual mesh filename=/home/yan/Documents/isaacsim_usd/FR5_V6/meshes/fr5_wsg50/FR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 scale=1. 1. 1.
- link FR5_link6: geometry collision mesh filename=/home/yan/Documents/isaacsim_usd/FR5_V6/meshes/fr5_wsg50/FR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 scale=1. 1. 1.; visual mesh filename=/home/yan/Documents/isaacsim_usd/FR5_V6/meshes/fr5_wsg50/FR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 scale=1. 1. 1.
- link base: geometry collision box size=0.146 0.05 0.072; collision cylinder length=0.018 radius=0.041

File: FR5_V6/urdf/rtq85.urdf (robot description, URDF)
Before this commit: robot robotiq_arg2f_85_model, 11 links, 10 joints
Links:
- removed link left_inner_finger_pad
- removed link right_inner_finger_pad
- removed link robotiq_arg2f_base_link
- added link robotiq_base_link, mass 0.22652; collision mesh filename=package://FR5_V6/meshes/rtq85/collision/robotiq_85_base_lin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; visual mesh filename=package://FR5_V6/meshes/rtq85/visual/robotiq_85_base_link.d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 scale=1.0 1.0 1.0
- link left_inner_finger: geometry collision mesh filename=package://FR5_V6/meshes/rtq85/collision/robotiq_85_finger_t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 scale=1.0 1.0 1.0; visual mesh filename=package://FR5_V6/meshes/rtq85/visual/robotiq_85_finger_tip_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 scale=1.0 1.0 1.0
- link left_inner_knuckle: geometry collision mesh filename=package://FR5_V6/meshes/rtq85/collision/robotiq_85_inner_kn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 scale=1.0 1.0 1.0; visual mesh filename=package://FR5_V6/meshes/rtq85/visual/robotiq_85_inner_knuck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 scale=1.0 1.0 1.0
- link left_outer_finger: geometry collision mesh filename=package://FR5_V6/meshes/rtq85/collision/robotiq_85_finger_l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 scale=1.0 1.0 1.0; visual mesh filename=package://FR5_V6/meshes/rtq85/visual/robotiq_85_finger_link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 scale=1.0 1.0 1.0
- link left_outer_knuckle: geometry collision mesh filename=package://FR5_V6/meshes/rtq85/collision/robotiq_85_outer_kn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 scale=1.0 1.0 1.0; visual mesh filename=package://FR5_V6/meshes/rtq85/visual/robotiq_85_outer_knuck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 scale=1.0 1.0 1.0
- link right_inner_finger: geometry collision mesh filename=package://FR5_V6/meshes/rtq85/collision/robotiq_85_finger_t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 scale=1.0 1.0 1.0; visual mesh filename=package://FR5_V6/meshes/rtq85/visual/robotiq_85_finger_tip_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 scale=1.0 1.0 1.0
- link right_inner_knuckle: geometry collision mesh filename=package://FR5_V6/meshes/rtq85/collision/robotiq_85_inner_kn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 scale=1.0 1.0 1.0; visual mesh filename=package://FR5_V6/meshes/rtq85/visual/robotiq_85_inner_knuck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 scale=1.0 1.0 1.0
- link right_outer_finger: geometry collision mesh filename=package://FR5_V6/meshes/rtq85/collision/robotiq_85_finger_l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 scale=1.0 1.0 1.0; visual mesh filename=package://FR5_V6/meshes/rtq85/visual/robotiq_85_finger_link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 scale=1.0 1.0 1.0
- link right_outer_knuckle: geometry collision mesh filename=package://FR5_V6/meshes/rtq85/collision/robotiq_85_outer_kn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 scale=1.0 1.0 1.0; visual mesh filename=package://FR5_V6/meshes/rtq85/visual/robotiq_85_outer_knuck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 scale=1.0 1.0 1.0
Joints:
- removed joint left_inner_finger_pad_joint
- removed joint right_inner_finger_pad_joint
- joint finger_joint: axis 1 0 0 -> 0 0 1; limit lower=0 upper=0.8 effort=1000 velocity=2.0 -> lower=0 upper=0.804 effort=1000 velocity=2.0; origin xyz=0 -0.0306011 0.054904 rpy=0 0 3.14159265359 -> xyz=0.05490451627 0.03060114443 0.0 rpy=3.14159265359 0.0 0.0; parent robotiq_arg2f_base_link -> robotiq_base_link
- joint left_inner_finger_joint: axis 1 0 0 -> 0 0 1; limit lower=-0.8757 upper=0 effort=1000 velocity=2.0 -> lower=-3.14 upper=3.14 effort=0.1 velocity=100.0; origin xyz=0 0.0061 0.0471 rpy=0 0 0 -> xyz=0.04303959807 -0.03759940821 0.0 rpy=0 0 0; parent left_outer_finger -> left_inner_knuckle; type revolute -> continuous
- joint left_inner_knuckle_joint: axis 1 0 0 -> 0 0 1; limit lower=0 upper=0.8757 effort=1000 velocity=2.0 -> lower=-3.14 upper=3.14 effort=0.1 velocity=100.0; origin xyz=0 -0.0127 0.06142 rpy=0 0 3.14159265359 -> xyz=0.06142 0.0127 0 rpy=3.14159265359 0 0; parent robotiq_arg2f_base_link -> robotiq_base_link; type revolute -> continuous
- joint left_outer_finger_joint: axis 1 0 0 -> (none); origin xyz=0 0.0315 -0.0041 rpy=0 0 0 -> xyz=-0.00408552455 -0.03148604435 0.0 rpy=0 0 0; type fixed -> continuous
- joint right_inner_finger_joint: axis 1 0 0 -> 0 0 1; limit lower=-0.8757 upper=0 effort=1000 velocity=2.0 -> lower=-3.14 upper=3.14 effort=0.1 velocity=100.0; origin xyz=0 0.0061 0.0471 rpy=0 0 0 -> xyz=0.04303959807 -0.03759940821 0.0 rpy=0 0 0; parent right_outer_finger -> right_inner_knuckle; type revolute -> continuous
- joint right_inner_knuckle_joint: axis 1 0 0 -> 0 0 1; limit lower=0 upper=0.8757 effort=1000 velocity=2.0 -> lower=-3.14 upper=3.14 effort=0.1 velocity=100.0; origin xyz=0 0.0127 0.06142 rpy=0 0 0.0 -> xyz=0.06142 -0.0127 0 rpy=0 0 0; parent robotiq_arg2f_base_link -> robotiq_base_link; type revolute -> continuous
- joint right_outer_finger_joint: axis 1 0 0 -> (none); origin xyz=0 0.0315 -0.0041 rpy=0 0 0 -> xyz=-0.00408552455 -0.03148604435 0.0 rpy=0 0 0; type fixed -> continuous
- joint right_outer_knuckle_joint: axis 1 0 0 -> 0 0 1; limit lower=0 upper=0.81 effort=1000 velocity=2.0 -> lower=-3.14 upper=3.14 effort=1000 velocity=100.0; origin xyz=0 0.0306011 0.054904 rpy=0 0 0 -> xyz=0.05490451627 -0.03060114443 0.0 rpy=0 0 0; parent robotiq_arg2f_base_link -> robotiq_base_link
